Commit message: Q2(b): vision-based look-at-point controller

File: ros2_iiwa/iiwa_description/gazebo/iiwa.gazebo.xacro (robot description, xacro)
@@ -14,8 +14,29 @@
       </plugin>
     </gazebo>
-    <!-- color -->
+    <!-- Link 7 appearance -->
     <gazebo reference="${prefix}link_7">
       <material>Gazebo/Gray</material>
     </gazebo>
+    <!-- Eye-in-hand camera sensor attached to camera_link -->
+    <gazebo reference="${prefix}camera_link">
+      <sensor name="eye_in_hand_camera" type="camera">
+        <pose>0 0 0 0 -0.922 -0.468</pose>
+        <always_on>true</always_on>
+        <update_rate>30</update_rate>
+        <topic>eye_in_hand_camera</topic>
+        <camera>
+          <horizontal_fov>1.047</horizontal_fov>
+          <image>
+            <width>640</width>
+            <height>480</height>
+            <format>R8G8B8</format>
+          </image>
+          <clip>
+            <near>0.02</near>
+            <far>10.0</far>
+          </clip>
+        </camera>
+      </sensor>
+    </gazebo>
   </xacro:macro>
 </robot>

File: ros2_iiwa/iiwa_description/urdf/iiwa.urdf.xacro (robot description, xacro)
@@ -170,4 +170,31 @@
   </link>
   <link name="${prefix}tool0"/>
+    <!-- Camera link rigidly attached to the end-effector -->
+  <link name="${prefix}camera_link">
+      <visual>
+        <origin xyz="0 0 0" rpy="0 0 0"/>
+        <geometry>
+          <box size="0.04 0.04 0.03"/>
+        </geometry>
+        <material name="gray"/>
+      </visual>
+      <collision>
+        <origin xyz="0 0 0" rpy="0 0 0"/>
+        <geometry>
+          <box size="0.04 0.04 0.03"/>
+        </geometry>
+      </collision>
+      <inertial>
+        <origin xyz="0 0 0" rpy="0 0 0"/>
+        <mass value="0.05"/>
+        <inertia
+          ixx="0.00001"
+          ixy="0.0"
+          ixz="0.0"
+          iyy="0.00001"
+          iyz="0.0"
+          izz="0.00001"/>
+      </inertial>
+  </link>
   <joint name="${prefix}joint_a1" type="revolute">
       <origin rpy="0 0 0" xyz="0 0 0"/>
@@ -225,4 +252,12 @@
       <axis xyz="0 0 0"/>
   </joint>
+    <!-- Fixed transform from iiwa link_7 to the eye-in-hand camera -->
+  <joint name="${prefix}camera_joint" type="fixed">
+      <parent link="${prefix}link_7"/>
+      <child link="${prefix}camera_link"/>
+      <origin
+        xyz="0 0 0.18"
+        rpy="0 0 0"/>
+  </joint>
   </xacro:macro>
 </robot>
